File: Circuit_Designs/Analog_Light_Project_Improved_Schematic.brd (EAGLE design)
At the start: 49.5 x 45.4 mm, 25 parts, among them IC1 4017D, T1 2N2222, T2 2N2222, T3 2N2222

Commit message: Improved PCB to be single-side
Parts:
- removed C4: 1µF, adafruit:C0805
- removed R1: 10k, adafruit:M0805
- removed R18: 330k, adafruit:M0805
- added C3: 1µF, rcl:C025-024X044
- added R2: 10k, rcl:0204/5
- added R3: (no value), rcl:0204/5
- C1: device adafruit:C0805 -> rcl:C025-024X044
- moved C1 1.80 mm to (21.6, 94.0)
- moved R11 1.27 mm to (15.2, 87.6)
- moved T3 1.27 mm to (25.4, 63.5)
- moved J1 1.27 mm to (16.5, 94.0)
Connections:
- net N$1: now also R3.2; no longer R18.2
- net N$12: now also R2.2; no longer R1.1
- net N$15: now also R2.1; no longer R1.2
- net N$2: now also C3.1; no longer C4.1
- net N$3: now also C3.2, R3.1; no longer C4.2, R18.1
Routing:
- net +9V: track 51.3 -> 61.7 mm, vias 2 -> 0
- net N$1: track 46.4 -> 54.7 mm, vias 2 -> 0
- net N$4: track 20.6 -> 26.9 mm, vias 1 -> 0
- net N$3: track 19.4 -> 16.1 mm
- net N$15: track 14.6 -> 13.0 mm
- net N$12: track 16.6 -> 15.3 mm
- net N$5: track 10.6 -> 10.1 mm
- net N$2: track 13.8 -> 13.3 mm
