File: Circuit_Designs/Analog_Light_Project_Improved_Schematic.sch (EAGLE design)
At the start: 25 parts, among them IC1 4017D, T1 2N2222, T2 2N2222, T3 2N2222

Commit message: Improved PCB to be single-side
Parts:
- removed C4: 1µF, adafruit:C-USC0805
- removed R1: 10k, adafruit:R-US_M0805
- removed R18: 330k, adafruit:R-US_M0805
- added C3: 1µF, rcl:C-US025-024X044
- added R2: 10k, rcl:R-US_0204/5
- added R3: (no value), rcl:R-US_0204/5
- C1: device adafruit:C-USC0805 -> rcl:C-US025-024X044
Connections:
- net N$1: now also R3.2; no longer R18.2
- net N$12: now also R2.2; no longer R1.1
- net N$15: now also R2.1; no longer R1.2
- net N$2: now also C3.1; no longer C4.1
- net N$3: now also C3.2, R3.1; no longer C4.2, R18.1
Other:
- moved on the sheet: T1
